File: input.kicad_sch (KiCad schematic)
At the start: 15 parts, among them J8 GPIO, U5 TLV3501AID

Commit message: rev. A for manufacturing
Parts:
- D3, D4: value UCLAMP3301D.TCT -> CDSOD323-T03; Current - Peak Pulse 10A (8/20µs) -> (none); DigiKey Part Number UCLAMP3301DCT-ND -> (none); MPN UCLAMP3301D.TCT -> CDSOD323-T03; Manufacturer Semtech Corporation -> BOURNS; TME Symbol UCLAMP3301D.TCT -> CDSOD323-T03; Voltage - Breakdown 3.5V -> (none); Voltage - Clamping 9.5V -> (none)
