File: jitter-hw.kicad_pcb (KiCad board)
At the start: 4 copper layers, 65 x 56 mm, 60 parts, among them J1 SWD Connector, J2 USB4105-GF-A-120, J3 USART Connector, J8 GPIO, SW1 B3U-1000P-B, U1 STM32H723VGT6, U2 ESDALC6V1W5, U3 AP2112K-3.3, U4 USBLC6-2SC6, U5 TLV3501AID, X1 25MHz/9pF

Commit message: rev. A for manufacturing
Parts:
- added G***: LOGO, LOGO, F.Cu at (144.2, 59.5)
Other:
- rule pad_to_mask_clearance: 0.1 -> 0
- board text added: "13/10/26 (Rev A) Łukasz Strama"
- board text removed: "10/04/26 (Rev A)"
