File: jitter-hw.kicad_sch (KiCad schematic)
At the start: 40 parts, among them J1 SWD Connector, J2 USB4105-GF-A-120, J3 USART Connector, SW1 B3U-1000P-B, U1 STM32H723VGT6, U2 ESDALC6V1W5, U3 AP2112K-3.3, U4 USBLC6-2SC6, X1 25MHz/9pF

Commit message: rev. A for manufacturing
Parts:
- D2: value UCLAMP3301D.TCT -> CDSOD323-T03; Current - Peak Pulse 10A (8/20µs) -> (none); DigiKey Part Number UCLAMP3301DCT-ND -> (none); MPN UCLAMP3301D.TCT -> CDSOD323-T03; Manufacturer Semtech Corporation -> BOURNS; TME Symbol UCLAMP3301D.TCT -> CDSOD323-T03; Voltage - Breakdown 3.5V -> (none); Voltage - Clamping 9.5V -> (none)
